File: hardware/curve-tracer.kicad_pcb (KiCad board)
At the start: 2 copper layers, 135 x 92 mm, 84 parts, among them J1 15V IN, J2 15V BENCH, J3 RANGE_FORCE, J4 RANGE_SENSE, J5 KELVIN HI / LO, J6 DUT G / D / S, J7 CN7 (morpho), J8 CN10 (morpho), Q1 BD139, Q2 MMBT3904, U1 OPA2197IDR, U2 OPA2197IDR, U3 OPA2197IDR

Commit message: hardware: J1 reverse-polarity P-FET, heatsink rule, NT2 justified
- Q3 HL2303 (JLC Preferred, -30 V, +/-20 V gate, <= 28.5 mV at 150 mA) in
  the high side of J1, with D6 (12 V gate-source clamp, D2's line) and R25
  (10k gate pull-down, Basic): no new loading fee. Placed in the free patch
  above J1; the +15V pour's left edge moves from x 12 to 17. No existing
  copper removed or moved, no Pass 1 copper involved. TP28 bare pad on VIN.
- check_topology.py asserts the protection and plants two new faults
  (drain/source swapped, gate Zener reversed): 55/55, 11/11 caught.
- DECISIONS.md: P-11 records the part choice and that the 9.06 V headroom
  is set downstream of the loop, so a Schottky would not have touched it;
  P-12 no EMI filter and why; P-13 no fiducials; NT2 stays, on the
  crossing numbers. J2 is not behind Q3 and is flagged.
- The heatsink is required for any short test: stated in README.md, an
  H4 verified item (tab isolation, case temperature), and silkscreen
  inside the keep-out where the heatsink covers it.
- Re-exported: ERC, DRC with schematic parity, and the checker are clean.

Co-Authored-By: Claude Opus 5.5 <noreply@anthropic.com>
Parts:
- added D6: BZT52C12 12V, Diode_SMD:D_SOD-123, F.Cu at (52.9, 44.4)
- added Q3: HL2303, Package_TO_SOT_SMD:SOT-23, F.Cu at (49.6, 44.9)
- added R25: 10k 1%, Resistor_SMD:R_0603_1608Metric, F.Cu at (55.4, 45.4)
- added TP28: VIN (pad), TestPoint:TestPoint_Pad_D1.0mm, F.Cu at (48.7, 41.8)
Connections:
- J1 pad 1: +15V -> /VIN
Routing:
- net /VIN: track 0.00 -> 14.3 mm
- net +15V: track 153.9 -> 163.3 mm
- net /RP_GATE: track 0.00 -> 5.27 mm
- net GNDPWR: track 9.99 -> 11.5 mm, vias 5 -> 6
Other:
- board text added: "BEFORE SHORT TEST"
- board text added: "FIT Q1 HEATSINK"
- board text added: "TAB = +15 V"

Commit message: hardware: label J2 polarity; design frozen pending the Oct 12 gate
J2 stays deliberately unprotected (DECISIONS.md P-14): it takes a bench
supply whose polarity is set and checked before connecting, unlike J1's
arbitrary wall adapter, which Q3 protects. Its pads now carry "+15V" and
"GND" in silkscreen. H4 adds a meter check of J2 polarity before first
power-up, and first power-up through J2 at a 100 mA limit, raised above
~120 mA before any held-short test.

Gerbers re-exported (front silkscreen only); DRC with schematic parity and
check_topology.py --self-test clean.

The design is frozen pending the Oct 12 stability gate.

Co-Authored-By: Claude Opus 5.5 <noreply@anthropic.com>
Other:
- board text added: "+15V"
- board text added: "GND"
Changed lines of the file:
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@@
+		)
+	)
+	(gr_text "+15V"
+		(at 45.6 70 0)
+		(layer "F.SilkS")
+		(effects
+			(font
+				(size 1.2 1.2)
+				(thickness 0.2)
+			)
+			(justify left)
+		)
+	)
+	(gr_text "GND"
+		(at 45.6 72.54 0)
+		(layer "F.SilkS")
+		(effects
+			(font
+				(size 1.2 1.2)
+				(thickness 0.2)
+			)
+			(justify left)
 		)
 	)

Commit message: Step 15 threshold 16 V; DUT-node design rule; D3 part number in schematic
- H4 step 15: pass <= 16.0 V (was 12.0 V). With D3 fitted, 13.3-14.8 V is
  the SMAJ12A working as specified; above 16 V is something other than the
  structural overshoot sim 10 predicts. D3 bounds a microsecond transient,
  not the 10 V ceiling; sustained overcurrent is the firmware limit's job.
  The scope is now centred at +10 V so a 16 V peak is on screen.
- Blueprint 3.3: everything on the DUT node is read as DUT current, with
  three instances (13's bridge, F-1's divider, D3's leakage). Anything
  added there is checked against range 3. 3.4 and F-1 point to it.
- D3 schematic and PCB fields: SMAJ12A, MDD, C113957, still DNP. Fields
  only; DRC with parity, ERC and the topology checker are clean.

Co-Authored-By: Claude Opus 5.5 <noreply@anthropic.com>
Parts:
- D3: value DNP (output clamp) -> SMAJ12A (DNP)
Changed lines of the file:
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@@
 			)
 		)
-		(property "Value" "DNP (output clamp)"
+		(property "Value" "SMAJ12A (DNP)"
 			(at 0 2.6 90)
 			(layer "F.Fab")
@@
 			)
 		)
-		(property "Description" "Output clamp footprint at DUT socket (§14.6)"
+		(property "Description" "Output clamp TVS at DUT socket; fit only if H4 step 15 fails (blueprint §3.6)"
 			(at 0 0 90)
 			(unlocked yes)
@@
 			)
 		)
-		(property "MPN" ""
+		(property "MPN" "SMAJ12A"
 			(at 0 0 90)
 			(layer "F.SilkS")
@@
 			)
 		)
-		(property "Manufacturer" ""
+		(property "Manufacturer" "MDD(Microdiode Semiconductor)"
 			(at 0 0 90)
 			(layer "F.SilkS")
@@
 			)
 		)
-		(property "LCSC" ""
+		(property "LCSC" "C113957"
 			(at 0 0 90)
 			(layer "F.SilkS")

Commit message: Fit D3 by default; step 15 verifies, step 13a tells D3 from no D3
- D3 SMAJ12A moves from DNP to PCBA: schematic, PCB, engineering BOM, JLC
  BOM and CPL (26 lines, 39 rows; +1 extended line, $54 in fees). Symbol
  is now Diode:SMAJ12A (unidirectional) instead of the bidirectional
  Device:D_TVS; pin 1, the cathode, stays on DUT_D. Gerbers unchanged.
- DECISIONS D3 records the trade: <= 1 uA on the DUT node, 10% of range 3
  full scale and negligible on range 1, with ranges 2-3 outside the MVP,
  against bounding the overshoot sim 10 predicts on every limit release.
- H4 step 15 is now a verification: expect 13.3-14.8 V, pass <= 16 V. It
  cannot confirm D3 on its own (the unclamped peak is also ~14.8 V), so new
  step 13a drives D3 into DC breakdown through 10 k from +15 V with J3 and
  the Kelvin pair off: 12.0-14.8 V means fitted and the right way round.
- check_topology: D3 polarity and fitted; the DUT-node parts list is
  fixed (blueprint 3.3). 59/59, 14 planted faults caught.
- C1, R4, R6, R8 values and descriptions filled, still DNP; C1 and R8 have
  MPN and LCSC. R4/R6 are on-hand generic parts with no MPN.

Co-Authored-By: Claude Opus 5.5 <noreply@anthropic.com>
Parts:
- C1: value DNP (C_f) -> 3.3p C0G (DNP)
- D3: value SMAJ12A (DNP) -> SMAJ12A
- R4: value DNP (R_B alt) -> 330 1% (DNP)
- R6: value DNP (R_sense alt) -> 10 1% (DNP)
- R8: value DNP (R_iso alt) -> 47 1% 1W (DNP)
Changed lines of the file:
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@@
 			)
 		)
-		(property "Value" "DNP (R_sense alt)"
+		(property "Value" "10 1% (DNP)"
 			(at 6.35 2.72 270)
 			(layer "F.Fab")
@@
 			)
 		)
-		(property "Description" "R_sense alternate-value footprint"
+		(property "Description" "R_sense alternate. 10 ohm axial IN PARALLEL with R5 = 5 ohm, only for a trip that reads low (CONTINGENCY.md §4). On hand, blueprint §8: no MPN"
 			(at 0 0 270)
 			(layer "F.Fab")
@@
 			)
 		)
-		(property "Value" "SMAJ12A (DNP)"
+		(property "Value" "SMAJ12A"
 			(at 0 2.6 90)
 			(layer "F.Fab")
@@
 			)
 		)
-		(property "Description" "Output clamp TVS at DUT socket; fit only if H4 step 15 fails (blueprint §3.6)"
+		(property "Description" "Output clamp TVS at DUT socket, fitted (blueprint §3.6)"
 			(at 0 0 90)
 			(unlocked yes)
@@
 			)
 		)
-		(property "Assembly" "DNP"
+		(property "Assembly" "PCBA"
 			(at 0 0 90)
 			(layer "F.SilkS")
@@
 			)
 		)
-		(attr smd dnp)
+		(attr smd)
 		(duplicate_pad_numbers_are_jumpers no)
 		(fp_line
@@
 			)
 		)
-		(property "Value" "DNP (C_f)"
+		(property "Value" "3.3p C0G (DNP)"
 			(at 0 1.43 0)
 			(layer "F.Fab")
@@
 			)
 		)
-		(property "Description" "C_f across R_f"
+		(property "Description" "C_f across R_f. 3.3 pF hand-fitted at H4 P3; the C_f sweep may change it (CONTINGENCY.md §2)"
 			(at 0 0 0)
 			(layer "F.Fab")
@@
 			)
 		)
-		(property "MPN" ""
+		(property "MPN" "0603CG3R3B500NT"
 			(at 0 0 0)
 			(layer "F.SilkS")
@@
 			)
 		)
-		(property "Manufacturer" ""
+		(property "Manufacturer" "FH (Guangdong Fenghua)"
 			(at 0 0 0)
 			(layer "F.SilkS")
@@
 			)
 		)
-		(property "LCSC" ""
+		(property "LCSC" "C2836771"
 			(at 0 0 0)
 			(layer "F.SilkS")
@@
 			)
 		)
-		(property "Value" "DNP (R_iso alt)"
+		(property "Value" "47 1% 1W (DNP)"
 			(at 6.35 2.72 270)
 			(layer "F.Fab")
@@
 			)
 		)
-		(property "Description" "R_iso alternate-value footprint"
+		(property "Description" "R_iso alternate. 47 ohm fitted ALONE, R7 removed first; in parallel it lowers R_iso (CONTINGENCY.md A6)"
 			(at 0 0 270)
 			(layer "F.Fab")
@@
 			)
 		)
-		(property "MPN" ""
+		(property "MPN" "RN1WS47ΩFT/BA1"
 			(at 0 0 270)
 			(layer "F.SilkS")
@@
 			)
 		)
-		(property "Manufacturer" ""
+		(property "Manufacturer" "TyoHM"
 			(at 0 0 270)
 			(layer "F.SilkS")
@@
 			)
 		)
-		(property "LCSC" ""
+		(property "LCSC" "C385394"
 			(at 0 0 270)
 			(layer "F.SilkS")
@@
 			)
 		)
-		(property "Value" "DNP (R_B alt)"
+		(property "Value" "330 1% (DNP)"
 			(at 6.35 2.72 90)
 			(layer "F.Fab")
@@
 			)
 		)
-		(property "Description" "R_B alternate-value footprint"
+		(property "Description" "R_B alternate. 330 ohm axial IN PARALLEL with R3 = 165 ohm (CONTINGENCY.md A5). On hand, blueprint §8: no MPN"
 			(at 0 0 90)
 			(layer "F.Fab")
